Commit message: Update rover.urdf.xacro

File: src/rover_description/urdf/rover.urdf.xacro (robot description, xacro)
@@ -66,5 +66,37 @@
         </visual>
     </link>
+    <link name="u_joint_2_link">
+        <visual>
+            <origin rpy="0 0 0" xyz="-175 239 -110"></origin>
+            <geometry>
+                <mesh filename="package://rover_description/meshes/u_joint.stl"></mesh>
+            </geometry>
+        </visual>
+    </link>
+    <link name="u_joint_3_link">
+        <visual>
+            <origin rpy="0 0 0" xyz="-175 239 -110"></origin>
+            <geometry>
+                <mesh filename="package://rover_description/meshes/u_joint.stl"></mesh>
+            </geometry>
+        </visual>
+    </link>
+    <link name="u_joint_4_link">
+        <visual>
+            <origin rpy="0 0 0" xyz="-175 239 -110"></origin>
+            <geometry>
+                <mesh filename="package://rover_description/meshes/u_joint.stl"></mesh>
+            </geometry>
+        </visual>
+    </link>
     <link name="u_joint_5_link">
+        <visual>
+            <origin rpy="0 0 0" xyz="-175 239 -110"></origin>
+            <geometry>
+                <mesh filename="package://rover_description/meshes/u_joint.stl"></mesh>
+            </geometry>
+        </visual>
+    </link>
+    <link name="u_joint_6_link">
         <visual>
             <origin rpy="0 0 0" xyz="-175 239 -110"></origin>
@@ -123,15 +155,43 @@
     <joint name="u_joint_1_joint" type="revolute">
         <axis xyz="0 0 1"></axis>
-        <limit lower="-1.57" upper="1.57" effort='10.0' velocity="1.0"></limit>
+        <limit lower="-0.785" upper="0.785" effort='10.0' velocity="1.0"></limit>
         <origin rpy="0 0 0" xyz="-80 0 0"></origin>
         <parent link="left_boogie_link"></parent>
         <child link="u_joint_1_link"></child>
     </joint>
+    <joint name="u_joint_2_joint" type="revolute">
+        <axis xyz="0 0 1"></axis>
+        <limit lower="-0.785" upper="0.785" effort='10.0' velocity="1.0"></limit>
+        <origin rpy="0 0 0" xyz="80 0 0"></origin>
+        <parent link="left_boogie_link"></parent>
+        <child link="u_joint_2_link"></child>
+    </joint>
+    <joint name="u_joint_3_joint" type="revolute">
+        <axis xyz="0 0 1"></axis>
+        <limit lower="-0.785" upper="0.785" effort='10.0' velocity="1.0"></limit>
+        <origin rpy="0 0 0" xyz="100 -5 -56"></origin>
+        <parent link="left_rocker_link"></parent>
+        <child link="u_joint_3_link"></child>
+    </joint>
+    <joint name="u_joint_4_joint" type="revolute">
+        <axis xyz="0 0 1"></axis>
+        <limit lower="-0.785" upper="0.785" effort='10.0' velocity="1.0"></limit>
+        <origin rpy="0 0 0" xyz="-80 0 0"></origin>
+        <parent link="right_boogie_link"></parent>
+        <child link="u_joint_4_link"></child>
+    </joint>
     <joint name="u_joint_5_joint" type="revolute">
         <axis xyz="0 0 1"></axis>
-        <limit lower="-1.57" upper="1.57" effort='10.0' velocity="1.0"></limit>
-        <origin rpy="0 0 0" xyz="80 0 0"></origin>
+        <limit lower="-0.785" upper="0.785" effort='10.0' velocity="1.0"></limit>
+        <origin rpy="0 0 0" xyz="80 0 -4"></origin>
         <parent link="right_boogie_link"></parent>
         <child link="u_joint_5_link"></child>
     </joint>
+    <joint name="u_joint_6_joint" type="revolute">
+        <axis xyz="0 0 1"></axis>
+        <limit lower="-0.785" upper="0.785" effort='10.0' velocity="1.0"></limit>
+        <origin rpy="0 0 0" xyz="100 2 -56"></origin>
+        <parent link="right_rocker_link"></parent>
+        <child link="u_joint_6_link"></child>
+    </joint>
 </robot>

Commit message: Update rover.urdf.xacro

File: src/rover_description/urdf/rover.urdf.xacro (robot description, xacro)
@@ -6,5 +6,5 @@
             <origin rpy="0 0 0" xyz="0 0 0"></origin>
             <geometry>
-                <mesh filename="package://rover_description/meshes/body_rover.stl"></mesh>
+                <mesh filename="package://rover_description/meshes/body_rover.stl" scale="0.001 0.001 0.001"></mesh>
             </geometry>
         </visual>
@@ -12,7 +12,7 @@
     <link name="left_leg_link">
         <visual>
-            <origin rpy ="0 0 0" xyz="-261 -10 -120"></origin>
-            <geometry>
-                <mesh filename="package://rover_description/meshes/leg_1.stl"></mesh>
+            <origin rpy="0 0 0" xyz="-0.261 -0.010 -0.120"></origin>
+            <geometry>
+                <mesh filename="package://rover_description/meshes/leg_1.stl" scale="0.001 0.001 0.001"></mesh>
             </geometry>
         </visual>
@@ -20,7 +20,7 @@
     <link name="right_leg_link">
         <visual>
-            <origin rpy="0 0 0" xyz="-261 -10 -120"></origin>
-            <geometry>
-                <mesh filename="package://rover_description/meshes/leg_1.stl"></mesh>
+            <origin rpy="0 0 0" xyz="-0.261 -0.010 -0.120"></origin>
+            <geometry>
+                <mesh filename="package://rover_description/meshes/leg_1.stl" scale="0.001 -0.001 0.001"></mesh>
             </geometry>
         </visual>
@@ -28,7 +28,7 @@
     <link name="left_rocker_link">
         <visual>
-            <origin rpy="0 0 0" xyz="-220 25 -120"></origin>
-            <geometry>
-                <mesh filename="package://rover_description/meshes/rocker_1.stl"></mesh>
+            <origin rpy="0 0 0" xyz="-0.220 0.025 -0.120"></origin>
+            <geometry>
+                <mesh filename="package://rover_description/meshes/rocker_1.stl" scale="0.001 0.001 0.001"></mesh>
             </geometry>
         </visual>
@@ -36,7 +36,7 @@
     <link name="right_rocker_link">
         <visual>
-            <origin rpy="0 0 0" xyz="-220 -25 -120"></origin>
-            <geometry>
-                <mesh filename="package://rover_description/meshes/rocker_1.stl" scale="1 -1 1"></mesh>
+            <origin rpy="0 0 0" xyz="-0.220 -0.025 -0.120"></origin>
+            <geometry>
+                <mesh filename="package://rover_description/meshes/rocker_1.stl" scale="0.001 -0.001 0.001"></mesh>
             </geometry>
         </visual>
@@ -44,7 +44,7 @@
     <link name="left_boogie_link">
         <visual>
-            <origin rpy="0 0 0" xyz="-80 0 -70"></origin>
-            <geometry>
-                <mesh filename="package://rover_description/meshes/boogie_1.stl"></mesh>
+            <origin rpy="0 0 0" xyz="-0.080 0.000 -0.070"></origin>
+            <geometry>
+                <mesh filename="package://rover_description/meshes/boogie_1.stl" scale="0.001 0.001 0.001"></mesh>
             </geometry>
         </visual>
@@ -52,7 +52,7 @@
     <link name="right_boogie_link">
         <visual>
-            <origin rpy="0 0 0" xyz="-80 0 -70"></origin>
-            <geometry>
-                <mesh filename="package://rover_description/meshes/boogie_1.stl" scale="1 -1 1"></mesh>
+            <origin rpy="0 0 0" xyz="-0.080 0.000 -0.070"></origin>
+            <geometry>
+                <mesh filename="package://rover_description/meshes/boogie_1.stl" scale="0.001 -0.001 0.001"></mesh>
             </geometry>
         </visual>
@@ -60,7 +60,7 @@
     <link name="u_joint_1_link">
         <visual>
-            <origin rpy="0 0 0" xyz="-175 239 -110"></origin>
-            <geometry>
-                <mesh filename="package://rover_description/meshes/u_joint.stl"></mesh>
+            <origin rpy="0 0 0" xyz="-0.175 0.239 -0.110"></origin>
+            <geometry>
+                <mesh filename="package://rover_description/meshes/u_joint.stl" scale="0.001 0.001 0.001"></mesh>
             </geometry>
         </visual>
@@ -68,7 +68,7 @@
     <link name="u_joint_2_link">
         <visual>
-            <origin rpy="0 0 0" xyz="-175 239 -110"></origin>
-            <geometry>
-                <mesh filename="package://rover_description/meshes/u_joint.stl"></mesh>
+            <origin rpy="0 0 0" xyz="-0.175 0.239 -0.110"></origin>
+            <geometry>
+                <mesh filename="package://rover_description/meshes/u_joint.stl" scale="0.001 0.001 0.001"></mesh>
             </geometry>
         </visual>
@@ -76,7 +76,7 @@
     <link name="u_joint_3_link">
         <visual>
-            <origin rpy="0 0 0" xyz="-175 239 -110"></origin>
-            <geometry>
-                <mesh filename="package://rover_description/meshes/u_joint.stl"></mesh>
+            <origin rpy="0 0 0" xyz="-0.175 0.239 -0.110"></origin>
+            <geometry>
+                <mesh filename="package://rover_description/meshes/u_joint.stl" scale="0.001 0.001 0.001"></mesh>
             </geometry>
         </visual>
@@ -84,7 +84,7 @@
     <link name="u_joint_4_link">
         <visual>
-            <origin rpy="0 0 0" xyz="-175 239 -110"></origin>
-            <geometry>
-                <mesh filename="package://rover_description/meshes/u_joint.stl"></mesh>
+            <origin rpy="0 0 0" xyz="-0.175 0.239 -0.110"></origin>
+            <geometry>
+                <mesh filename="package://rover_description/meshes/u_joint.stl" scale="0.001 0.001 0.001"></mesh>
             </geometry>
         </visual>
@@ -92,7 +92,7 @@
     <link name="u_joint_5_link">
         <visual>
-            <origin rpy="0 0 0" xyz="-175 239 -110"></origin>
-            <geometry>
-                <mesh filename="package://rover_description/meshes/u_joint.stl"></mesh>
+            <origin rpy="0 0 0" xyz="-0.175 0.239 -0.110"></origin>
+            <geometry>
+                <mesh filename="package://rover_description/meshes/u_joint.stl" scale="0.001 0.001 0.001"></mesh>
             </geometry>
         </visual>
@@ -100,12 +100,60 @@
     <link name="u_joint_6_link">
         <visual>
-            <origin rpy="0 0 0" xyz="-175 239 -110"></origin>
-            <geometry>
-                <mesh filename="package://rover_description/meshes/u_joint.stl"></mesh>
+            <origin rpy="0 0 0" xyz="-0.175 0.239 -0.110"></origin>
+            <geometry>
+                <mesh filename="package://rover_description/meshes/u_joint.stl" scale="0.001 0.001 0.001"></mesh>
+            </geometry>
+        </visual>
+    </link>
+    <link name="wheel_1_link">
+        <visual>
+            <origin rpy="0 0 0" xyz="0 0 0"></origin>
+            <geometry>
+                <mesh filename="package://rover_description/meshes/wheel.stl" scale="0.001 -0.001 0.001"></mesh>
+            </geometry>
+        </visual>
+    </link>
+    <link name="wheel_2_link">
+        <visual>
+            <origin rpy="0 0 0" xyz="0 0 0"></origin>
+            <geometry>
+                <mesh filename="package://rover_description/meshes/wheel.stl" scale="0.001 -0.001 0.001"></mesh>
+            </geometry>
+        </visual>
+    </link>
+    <link name="wheel_3_link">
+        <visual>
+            <origin rpy="0 0 0" xyz="0 0 0"></origin>
+            <geometry>
+                <mesh filename="package://rover_description/meshes/wheel.stl" scale="0.001 -0.001 0.001"></mesh>
+            </geometry>
+        </visual>
+    </link>
+    <link name="wheel_4_link">
+        <visual>
+            <origin rpy="0 0 0" xyz="0 0 0"></origin>
+            <geometry>
+                <mesh filename="package://rover_description/meshes/wheel.stl" scale="0.001 -0.001 0.001"></mesh>
+            </geometry>
+        </visual>
+    </link>
+    <link name="wheel_5_link">
+        <visual>
+            <origin rpy="0 0 0" xyz="0 0 0"></origin>
+            <geometry>
+                <mesh filename="package://rover_description/meshes/wheel.stl" scale="0.001 -0.001 0.001"></mesh>
+            </geometry>
+        </visual>
+    </link>
+    <link name="wheel_6_link">
+        <visual>
+            <origin rpy="0 0 0" xyz="0 0 0"></origin>
+            <geometry>
+                <mesh filename="package://rover_description/meshes/wheel.stl" scale="0.001 -0.001 0.001"></mesh>
             </geometry>
         </visual>
     </link>
     <joint name="base_part_link_joint" type="fixed">
-        <origin rpy="0 0 0" xyz="-183 -75 -118"></origin>
+        <origin rpy="0 0 0" xyz="-0.183 -0.075 -0.118"></origin>
         <parent link="base_link"></parent>
         <child link="base_part_link"></child>
@@ -114,5 +162,5 @@
         <axis xyz="0 1 0"></axis>
         <limit lower="-1.57" upper="1.57" effort='10.0' velocity="1.0"></limit>
-        <origin rpy="0 0 0" xyz="0 -105 0"></origin>
+        <origin rpy="0 0 0" xyz="0 -0.105 0"></origin>
         <parent link="base_link"></parent>
         <child link="left_leg_link"></child>
@@ -121,5 +169,5 @@
         <axis xyz="0 1 0"></axis>
         <limit lower="-1.57" upper="1.57" effort='10.0' velocity="1.0"></limit>
-        <origin rpy="0 0 0" xyz="0 120 0"></origin>
+        <origin rpy="0 0 0" xyz="0 0.120 0"></origin>
         <parent link="base_link"></parent>
         <child link="right_leg_link"></child>
@@ -128,5 +176,5 @@
         <axis xyz="0 1 0"></axis>
         <limit lower="-1.04" upper="1.04" effort='10.0' velocity="1.0"></limit>
-        <origin rpy="0 0 0" xyz="0 -129 0"></origin>
+        <origin rpy="0 0 0" xyz="0 -0.129 0"></origin>
         <parent link="base_link"></parent>
         <child link="left_rocker_link"></child>
@@ -135,5 +183,5 @@
         <axis xyz="0 1 0"></axis>
         <limit lower="-1.04" upper="1.04" effort='10.0' velocity="1.0"></limit>
-        <origin rpy="0 0 0" xyz="0 129 0"></origin>
+        <origin rpy="0 0 0" xyz="0 0.129 0"></origin>
         <parent link="base_link"></parent>
         <child link="right_rocker_link"></child>
@@ -142,5 +190,5 @@
         <axis xyz="0 1 0"></axis>
         <limit lower="-1.57" upper="1.57" effort='10.0' velocity="1.0"></limit>
-        <origin rpy="0 0 0" xyz="-183 -27 -50"></origin>
+        <origin rpy="0 0 0" xyz="-0.183 -0.027 -0.050"></origin>
         <parent link="left_leg_link"></parent>
         <child link="left_boogie_link"></child>
@@ -149,5 +197,5 @@
         <axis xyz="0 1 0"></axis>
         <limit lower="-1.57" upper="1.57" effort='10.0' velocity="1.0"></limit>
-        <origin rpy="0 0 0" xyz="-183 5 -50"></origin>
+        <origin rpy="0 0 0" xyz="-0.183 0.005 -0.050"></origin>
         <parent link="right_leg_link"></parent>
         <child link="right_boogie_link"></child>
@@ -156,5 +204,5 @@
         <axis xyz="0 0 1"></axis>
         <limit lower="-0.785" upper="0.785" effort='10.0' velocity="1.0"></limit>
-        <origin rpy="0 0 0" xyz="-80 0 0"></origin>
+        <origin rpy="0 0 0" xyz="-0.080 0 0"></origin>
         <parent link="left_boogie_link"></parent>
         <child link="u_joint_1_link"></child>
@@ -163,5 +211,5 @@
         <axis xyz="0 0 1"></axis>
         <limit lower="-0.785" upper="0.785" effort='10.0' velocity="1.0"></limit>
-        <origin rpy="0 0 0" xyz="80 0 0"></origin>
+        <origin rpy="0 0 0" xyz="0.080 0 0"></origin>
         <parent link="left_boogie_link"></parent>
         <child link="u_joint_2_link"></child>
@@ -170,5 +218,5 @@
         <axis xyz="0 0 1"></axis>
         <limit lower="-0.785" upper="0.785" effort='10.0' velocity="1.0"></limit>
-        <origin rpy="0 0 0" xyz="100 -5 -56"></origin>
+        <origin rpy="0 0 0" xyz="0.100 -0.005 -0.056"></origin>
         <parent link="left_rocker_link"></parent>
         <child link="u_joint_3_link"></child>
@@ -177,5 +225,5 @@
         <axis xyz="0 0 1"></axis>
         <limit lower="-0.785" upper="0.785" effort='10.0' velocity="1.0"></limit>
-        <origin rpy="0 0 0" xyz="-80 0 0"></origin>
+        <origin rpy="0 0 0" xyz="-0.080 0 0"></origin>
         <parent link="right_boogie_link"></parent>
         <child link="u_joint_4_link"></child>
@@ -184,5 +232,5 @@
         <axis xyz="0 0 1"></axis>
         <limit lower="-0.785" upper="0.785" effort='10.0' velocity="1.0"></limit>
-        <origin rpy="0 0 0" xyz="80 0 -4"></origin>
+        <origin rpy="0 0 0" xyz="0.080 0 -0.004"></origin>
         <parent link="right_boogie_link"></parent>
         <child link="u_joint_5_link"></child>
@@ -191,7 +239,43 @@
         <axis xyz="0 0 1"></axis>
         <limit lower="-0.785" upper="0.785" effort='10.0' velocity="1.0"></limit>
-        <origin rpy="0 0 0" xyz="100 2 -56"></origin>
+        <origin rpy="0 0 0" xyz="0.100 0.002 -0.056"></origin>
         <parent link="right_rocker_link"></parent>
         <child link="u_joint_6_link"></child>
     </joint>
+    <joint name="wheel_1_joint" type="continuous">
+        <axis xyz="0 1 0"></axis>
+        <origin rpy="0 0 0" xyz="0 -0.019 -0.065"></origin>
+        <parent link="u_joint_1_link"></parent>
+        <child link="wheel_1_link"></child>
+    </joint>
+    <joint name="wheel_2_joint" type="continuous">
+        <axis xyz="0 1 0"></axis>
+        <origin rpy="0 0 0" xyz="0 -0.019 -0.065"></origin>
+        <parent link="u_joint_2_link"></parent>
+        <child link="wheel_2_link"></child>
+    </joint>
+    <joint name="wheel_3_joint" type="continuous">
+        <axis xyz="0 1 0"></axis>
+        <origin rpy="0 0 0" xyz="0 -0.019 -0.065"></origin>
+        <parent link="u_joint_3_link"></parent>
+        <child link="wheel_3_link"></child>
+    </joint>
+    <joint name="wheel_4_joint" type="continuous">
+        <axis xyz="0 1 0"></axis>
+        <origin rpy="0 0 0" xyz="0 -0.019 -0.065"></origin>
+        <parent link="u_joint_4_link"></parent>
+        <child link="wheel_4_link"></child>
+    </joint>
+    <joint name="wheel_5_joint" type="continuous">
+        <axis xyz="0 1 0"></axis>
+        <origin rpy="0 0 0" xyz="0 -0.019 -0.065"></origin>
+        <parent link="u_joint_5_link"></parent>
+        <child link="wheel_5_link"></child>
+    </joint>
+    <joint name="wheel_6_joint" type="continuous">
+        <axis xyz="0 1 0"></axis>
+        <origin rpy="0 0 0" xyz="0 -0.019 -0.065"></origin>
+        <parent link="u_joint_6_link"></parent>
+        <child link="wheel_6_link"></child>
+    </joint>
 </robot>
