Commit message: Add files via upload

File: src/rover_description/urdf/rover.urdf.xacro (robot description, xacro)
@@ -1,14 +1,30 @@
 <?xml version="1.0"?>
-<robot name="rover">
+<robot xmlns:xacro="http://www.ros.org/wiki/xacro" name="rover">
     <link name="base_link"></link>
     <link name="base_part_link">
-        <visual>
-            <origin rpy="0 0 0" xyz="0 0 0"></origin>
+        <inertial>
+            <origin xyz="0.36858011704103055 0.12727195552741655 0.2893761824201176" rpy="0 0 0"/>
+            <mass value="5.3148472840078265"/>
+            <inertia ixx="0.035413" iyy="0.043631" izz="0.066908" ixy="0.000486" iyz="-0.000133" ixz="0.001263"/>
+          </inertial>
+        <visual>
+            <origin rpy="0 0 0" xyz="0 0 0"/>
             <geometry>
                 <mesh filename="package://rover_description/meshes/body_rover.stl" scale="0.001 0.001 0.001"></mesh>
             </geometry>
         </visual>
+        <collision>
+            <origin rpy="0 0 0" xyz="0 0 0.5"/>
+            <geometry>
+                <mesh filename="package://rover_description/meshes/body_rover.stl" scale="0.001 0.001 0.001"></mesh>
+            </geometry>
+        </collision>
     </link>
     <link name="left_leg_link">
+        <inertial>
+            <origin xyz="0.0940898084139219 0.012814069160764302 -0.012373797524457275" rpy="0 0 0"/>
+            <mass value="0.6560655147003178"/>
+            <inertia ixx="0.00059" iyy="0.004256" izz="0.003752" ixy="-2e-06" iyz="6e-06" ixz="0.001033"/>
+          </inertial>
         <visual>
             <origin rpy="0 0 0" xyz="-0.261 -0.010 -0.120"></origin>
@@ -17,6 +33,17 @@
             </geometry>
         </visual>
+        <collision>
+            <origin rpy="0 0 0" xyz="-0.261 -0.010 -0.120"></origin>
+            <geometry>
+                <mesh filename="package://rover_description/meshes/leg_1.stl" scale="0.001 0.001 0.001"></mesh>
+            </geometry>
+        </collision>
     </link>
     <link name="right_leg_link">
+        <inertial>
+            <origin xyz="0.09408981018832419 -0.012814870490642113 -0.012373814218106793" rpy="0 0 0"/>
+            <mass value="0.6560656136558927"/>
+            <inertia ixx="0.00059" iyy="0.004256" izz="0.003752" ixy="2e-06" iyz="-6e-06" ixz="0.001033"/>
+          </inertial>
         <visual>
             <origin rpy="0 0 0" xyz="-0.261 -0.010 -0.120"></origin>
@@ -25,6 +52,17 @@
             </geometry>
         </visual>
+        <collision>
+            <origin rpy="0 0 0" xyz="-0.261 -0.010 -0.120"></origin>
+            <geometry>
+                <mesh filename="package://rover_description/meshes/leg_1.stl" scale="0.001 -0.001 0.001"></mesh>
+            </geometry>
+        </collision>
     </link>
     <link name="left_rocker_link">
+        <inertial>
+            <origin xyz="-0.06571336847368092 -0.013275152182515076 -0.055118178975015475" rpy="0 0 0"/>
+            <mass value="0.8937260483050995"/>
+            <inertia ixx="0.002073" iyy="0.003258" izz="0.001843" ixy="-2.3e-05" iyz="-7.1e-05" ixz="-0.001236"/>
+        </inertial>
         <visual>
             <origin rpy="0 0 0" xyz="-0.220 0.025 -0.120"></origin>
@@ -33,6 +71,17 @@
             </geometry>
         </visual>
+        <collision>
+            <origin rpy="0 0 0" xyz="-0.220 0.025 -0.120"></origin>
+            <geometry>
+                <mesh filename="package://rover_description/meshes/rocker_1.stl" scale="0.001 0.001 0.001"></mesh>
+            </geometry>
+        </collision>
     </link>
     <link name="right_rocker_link">
+        <inertial>
+            <origin xyz="-0.0656809601110295 0.013042069644830123 -0.054335275342790645" rpy="0 0 0"/>
+            <mass value="0.9511150507226518"/>
+            <inertia ixx="0.002083" iyy="0.003269" izz="0.001848" ixy="1.6e-05" iyz="-3.7e-05" ixz="-0.001236"/>
+          </inertial>
         <visual>
             <origin rpy="0 0 0" xyz="-0.220 -0.025 -0.120"></origin>
@@ -41,6 +90,17 @@
             </geometry>
         </visual>
+        <collision>
+            <origin rpy="0 0 0" xyz="-0.220 -0.025 -0.120"></origin>
+            <geometry>
+                <mesh filename="package://rover_description/meshes/rocker_1.stl" scale="0.001 -0.001 0.001"></mesh>
+            </geometry>
+        </collision>
     </link>
     <link name="left_boogie_link">
+        <inertial>
+            <origin xyz="-2.773434771169425e-05 0.01378851335933029 -0.019093045660989794" rpy="0 0 0"/>
+            <mass value="1.4914158227201482"/>
+            <inertia ixx="0.002319" iyy="0.009171" izz="0.00813" ixy="-7e-06" iyz="-0.000106" ixz="6e-06"/>
+          </inertial>
         <visual>
             <origin rpy="0 0 0" xyz="-0.080 0.000 -0.070"></origin>
@@ -49,6 +109,17 @@
             </geometry>
         </visual>
+        <collision>
+            <origin rpy="0 0 0" xyz="-0.080 0.000 -0.070"></origin>
+            <geometry>
+                <mesh filename="package://rover_description/meshes/boogie_1.stl" scale="0.001 0.001 0.001"></mesh>
+            </geometry>
+        </collision>
     </link>
     <link name="right_boogie_link">
+        <inertial>
+            <origin xyz="8.210657408652677e-05 -0.013101623219513326 -0.01912358611502865" rpy="0 0 0"/>
+            <mass value="1.4914778130132003"/>
+            <inertia ixx="0.00232" iyy="0.009173" izz="0.008131" ixy="0.0" iyz="-0.000101" ixz="-1e-06"/>
+          </inertial>
         <visual>
             <origin rpy="0 0 0" xyz="-0.080 0.000 -0.070"></origin>
@@ -57,186 +128,420 @@
             </geometry>
         </visual>
+        <collision>
+            <origin rpy="0 0 0" xyz="-0.080 0.000 -0.070"></origin>
+            <geometry>
+                <mesh filename="package://rover_description/meshes/boogie_1.stl" scale="0.001 -0.001 0.001"></mesh>
+            </geometry>
+        </collision>
     </link>
     <link name="u_joint_1_link">
-        <visual>
-            <origin rpy="0 0 0" xyz="-0.175 0.239 -0.110"></origin>
-            <geometry>
-                <mesh filename="package://rover_description/meshes/u_joint.stl" scale="0.001 0.001 0.001"></mesh>
-            </geometry>
-        </visual>
+        <inertial>
+            <origin xyz="8.210657408652677e-05 -0.013101623219513326 -0.01912358611502865" rpy="0 0 0"/>
+            <mass value="1.4914778130132003"/>
+            <inertia ixx="0.00232" iyy="0.009173" izz="0.008131" ixy="0.0" iyz="-0.000101" ixz="-1e-06"/>
+          </inertial>
+        <visual>
+            <origin rpy="0 0 0" xyz="-0.175 0.239 -0.110"></origin>
+            <geometry>
+                <mesh filename="package://rover_description/meshes/u_joint.stl" scale="0.001 0.001 0.001"></mesh>
+            </geometry>
+        </visual>
+        <collision>
+            <origin rpy="0 0 0" xyz="-0.175 0.239 -0.110"></origin>
+            <geometry>
+                <mesh filename="package://rover_description/meshes/u_joint.stl" scale="0.001 0.001 0.001"></mesh>
+            </geometry>
+        </collision>
     </link>
     <link name="u_joint_2_link">
-        <visual>
-            <origin rpy="0 0 0" xyz="-0.175 0.239 -0.110"></origin>
-            <geometry>
-                <mesh filename="package://rover_description/meshes/u_joint.stl" scale="0.001 0.001 0.001"></mesh>
-            </geometry>
-        </visual>
+        <inertial>
+            <origin xyz="8.210657408652677e-05 -0.013101623219513326 -0.01912358611502865" rpy="0 0 0"/>
+            <mass value="1.4914778130132003"/>
+            <inertia ixx="0.00232" iyy="0.009173" izz="0.008131" ixy="0.0" iyz="-0.000101" ixz="-1e-06"/>
+          </inertial>
+        <visual>
+            <origin rpy="0 0 0" xyz="-0.175 0.239 -0.110"></origin>
+            <geometry>
+                <mesh filename="package://rover_description/meshes/u_joint.stl" scale="0.001 0.001 0.001"></mesh>
+            </geometry>
+        </visual>
+        <collision>
+            <origin rpy="0 0 0" xyz="-0.175 0.239 -0.110"></origin>
+            <geometry>
+                <mesh filename="package://rover_description/meshes/u_joint.stl" scale="0.001 0.001 0.001"></mesh>
+            </geometry>
+        </collision>
     </link>
     <link name="u_joint_3_link">
-        <visual>
-            <origin rpy="0 0 0" xyz="-0.175 0.239 -0.110"></origin>
-            <geometry>
-                <mesh filename="package://rover_description/meshes/u_joint.stl" scale="0.001 0.001 0.001"></mesh>
-            </geometry>
-        </visual>
+        <inertial>
+            <origin xyz="8.210657408652677e-05 -0.013101623219513326 -0.01912358611502865" rpy="0 0 0"/>
+            <mass value="1.4914778130132003"/>
+            <inertia ixx="0.00232" iyy="0.009173" izz="0.008131" ixy="0.0" iyz="-0.000101" ixz="-1e-06"/>
+          </inertial>
+        <visual>
+            <origin rpy="0 0 0" xyz="-0.175 0.239 -0.110"></origin>
+            <geometry>
+                <mesh filename="package://rover_description/meshes/u_joint.stl" scale="0.001 0.001 0.001"></mesh>
+            </geometry>
+        </visual>
+        <collision>
+            <origin rpy="0 0 0" xyz="-0.175 0.239 -0.110"></origin>
+            <geometry>
+                <mesh filename="package://rover_description/meshes/u_joint.stl" scale="0.001 0.001 0.001"></mesh>
+            </geometry>
+        </collision>
     </link>
     <link name="u_joint_4_link">
-        <visual>
-            <origin rpy="0 0 0" xyz="-0.175 0.239 -0.110"></origin>
-            <geometry>
-                <mesh filename="package://rover_description/meshes/u_joint.stl" scale="0.001 0.001 0.001"></mesh>
-            </geometry>
-        </visual>
+        <inertial>
+            <origin xyz="8.210657408652677e-05 -0.013101623219513326 -0.01912358611502865" rpy="0 0 0"/>
+            <mass value="1.4914778130132003"/>
+            <inertia ixx="0.00232" iyy="0.009173" izz="0.008131" ixy="0.0" iyz="-0.000101" ixz="-1e-06"/>
+          </inertial>
+        <visual>
+            <origin rpy="0 0 0" xyz="-0.175 0.239 -0.110"></origin>
+            <geometry>
+                <mesh filename="package://rover_description/meshes/u_joint.stl" scale="0.001 0.001 0.001"></mesh>
+            </geometry>
+        </visual>
+        <collision>
+            <origin rpy="0 0 0" xyz="-0.175 0.239 -0.110"></origin>
+            <geometry>
+                <mesh filename="package://rover_description/meshes/u_joint.stl" scale="0.001 0.001 0.001"></mesh>
+            </geometry>
+        </collision>
     </link>
     <link name="u_joint_5_link">
-        <visual>
-            <origin rpy="0 0 0" xyz="-0.175 0.239 -0.110"></origin>
-            <geometry>
-                <mesh filename="package://rover_description/meshes/u_joint.stl" scale="0.001 0.001 0.001"></mesh>
-            </geometry>
-        </visual>
+        <inertial>
+            <origin xyz="8.210657408652677e-05 -0.013101623219513326 -0.01912358611502865" rpy="0 0 0"/>
+            <mass value="1.4914778130132003"/>
+            <inertia ixx="0.00232" iyy="0.009173" izz="0.008131" ixy="0.0" iyz="-0.000101" ixz="-1e-06"/>
+          </inertial>
+        <visual>
+            <origin rpy="0 0 0" xyz="-0.175 0.239 -0.110"></origin>
+            <geometry>
+                <mesh filename="package://rover_description/meshes/u_joint.stl" scale="0.001 0.001 0.001"></mesh>
+            </geometry>
+        </visual>
+        <collision>
+            <origin rpy="0 0 0" xyz="-0.175 0.239 -0.110"></origin>
+            <geometry>
+                <mesh filename="package://rover_description/meshes/u_joint.stl" scale="0.001 0.001 0.001"></mesh>
+            </geometry>
+        </collision>
     </link>
     <link name="u_joint_6_link">
-        <visual>
-            <origin rpy="0 0 0" xyz="-0.175 0.239 -0.110"></origin>
-            <geometry>
-                <mesh filename="package://rover_description/meshes/u_joint.stl" scale="0.001 0.001 0.001"></mesh>
-            </geometry>
-        </visual>
+        <inertial>
+            <origin xyz="8.210657408652677e-05 -0.013101623219513326 -0.01912358611502865" rpy="0 0 0"/>
+            <mass value="1.4914778130132003"/>
+            <inertia ixx="0.00232" iyy="0.009173" izz="0.008131" ixy="0.0" iyz="-0.000101" ixz="-1e-06"/>
+          </inertial>
+        <visual>
+            <origin rpy="0 0 0" xyz="-0.175 0.239 -0.110"></origin>
+            <geometry>
+                <mesh filename="package://rover_description/meshes/u_joint.stl" scale="0.001 0.001 0.001"></mesh>
+            </geometry>
+        </visual>
+        <collision>
+            <origin rpy="0 0 0" xyz="-0.175 0.239 -0.110"></origin>
+            <geometry>
+                <mesh filename="package://rover_description/meshes/u_joint.stl" scale="0.001 0.001 0.001"></mesh>
+            </geometry>
+        </collision>
     </link>
     <link name="wheel_1_link">
-        <visual>
-            <origin rpy="0 0 0" xyz="0 0 0"></origin>
-            <geometry>
-                <mesh filename="package://rover_description/meshes/wheel.stl" scale="0.001 -0.001 0.001"></mesh>
-            </geometry>
-        </visual>
+        <inertial>
+            <origin xyz="-1.0959477414473895e-07 -0.035645342277154296 3.2835295757371874e-07" rpy="0 0 0"/>
+            <mass value="0.33507957881433253"/>
+            <inertia ixx="0.000264" iyy="0.000363" izz="0.000264" ixy="-0.0" iyz="0.0" ixz="-0.0"/>
+          </inertial>
+        <visual>
+            <origin rpy="0 0 0" xyz="0 0 0"></origin>
+            <geometry>
+                <mesh filename="package://rover_description/meshes/wheel.stl" scale="0.001 -0.001 0.001"></mesh>
+            </geometry>
+        </visual>
+        <collision>
+            <origin rpy="0 0 0" xyz="0 0 0"></origin>
+            <geometry>
+                <mesh filename="package://rover_description/meshes/wheel.stl" scale="0.001 -0.001 0.001"></mesh>
+            </geometry>
+            <gazebo>
+                <surface>
+                    <friction>
+                        <ode>
+                            <mu>5.0</mu>      <!-- Friction coefficient -->
+                            <mu2>5.0</mu2>    <!-- Lateral friction coefficient -->
+                        </ode>
+                    </friction>
+                    <bounce>
+                        <restitution_coefficient>0.0</restitution_coefficient>
+                        <threshold>1000.0</threshold>
+                    </bounce>
+                    <contact>
+                        <ode>
+                            <kp>100000.0</kp> <!-- Stiffness parameter -->
+                            <kd>1.0</kd>      <!-- Damping parameter -->
+                        </ode>
+                    </contact>
+                </surface>
+            </gazebo>
+        </collision>
     </link>
     <link name="wheel_2_link">
-        <visual>
-            <origin rpy="0 0 0" xyz="0 0 0"></origin>
-            <geometry>
-                <mesh filename="package://rover_description/meshes/wheel.stl" scale="0.001 -0.001 0.001"></mesh>
-            </geometry>
-        </visual>
+        <inertial>
+            <origin xyz="-1.0959477414473895e-07 -0.035645342277154296 3.2835295757371874e-07" rpy="0 0 0"/>
+            <mass value="0.33507957881433253"/>
+            <inertia ixx="0.000264" iyy="0.000363" izz="0.000264" ixy="-0.0" iyz="0.0" ixz="-0.0"/>
+          </inertial>
+        <visual>
+            <origin rpy="0 0 0" xyz="0 0 0"></origin>
+            <geometry>
+                <mesh filename="package://rover_description/meshes/wheel.stl" scale="0.001 -0.001 0.001"></mesh>
+            </geometry>
+        </visual>
+        <collision>
+            <origin rpy="0 0 0" xyz="0 0 0"></origin>
+            <geometry>
+                <mesh filename="package://rover_description/meshes/wheel.stl" scale="0.001 -0.001 0.001"></mesh>
+            </geometry>
+            <gazebo>
+                <surface>
+                    <friction>
+                        <ode>
+                            <mu>5.0</mu>      <!-- Friction coefficient -->
+                            <mu2>5.0</mu2>    <!-- Lateral friction coefficient -->
+                        </ode>
+                    </friction>
+                    <bounce>
+                        <restitution_coefficient>0.0</restitution_coefficient>
+                        <threshold>1000.0</threshold>
+                    </bounce>
+                    <contact>
+                        <ode>
+                            <kp>100000.0</kp> <!-- Stiffness parameter -->
+                            <kd>1.0</kd>      <!-- Damping parameter -->
+                        </ode>
+                    </contact>
+                </surface>
+            </gazebo>
+        </collision>
     </link>
     <link name="wheel_3_link">
-        <visual>
-            <origin rpy="0 0 0" xyz="0 0 0"></origin>
-            <geometry>
-                <mesh filename="package://rover_description/meshes/wheel.stl" scale="0.001 -0.001 0.001"></mesh>
-            </geometry>
-        </visual>
+        <inertial>
+            <origin xyz="-1.0959477414473895e-07 -0.035645342277154296 3.2835295757371874e-07" rpy="0 0 0"/>
+            <mass value="0.33507957881433253"/>
+            <inertia ixx="0.000264" iyy="0.000363" izz="0.000264" ixy="-0.0" iyz="0.0" ixz="-0.0"/>
+          </inertial>
+        <visual>
+            <origin rpy="0 0 0" xyz="0 0 0"></origin>
+            <geometry>
+                <mesh filename="package://rover_description/meshes/wheel.stl" scale="0.001 -0.001 0.001"></mesh>
+            </geometry>
+        </visual>
+        <collision>
+            <origin rpy="0 0 0" xyz="0 0 0"></origin>
+            <geometry>
+                <mesh filename="package://rover_description/meshes/wheel.stl" scale="0.001 -0.001 0.001"></mesh>
+            </geometry>
+            <gazebo>
+                <surface>
+                    <friction>
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