Commit message: Add files via upload

File: src/rover_description/urdf/rover.urdf.xacro (robot description, xacro)
@@ -549,5 +549,5 @@
     </joint>
     <joint name="wheel_1_joint" type="continuous">
-        <axis xyz="0 1 0"></axis>
+        <axis xyz="0 -1 0"></axis>
         <origin rpy="0 0 0" xyz="0 -0.019 -0.065"></origin>
         <parent link="u_joint_1_link"></parent>
@@ -573,5 +573,5 @@
     </joint>
     <joint name="wheel_4_joint" type="continuous">
-        <axis xyz="0 1 0"></axis>
+        <axis xyz="0 -1 0"></axis>
         <origin rpy="0 0 0" xyz="0 -0.019 -0.065"></origin>
         <parent link="u_joint_4_link"></parent>
@@ -596,5 +596,70 @@
         <velocity>0.0</velocity> <!-- Ensure no initial velocity -->
     </joint>
-    <gazebo>
+  <!-- LIDAR -->
+  <xacro:macro name="inertial_cylinder" params="mass length radius *origin">
+    <inertial>
+        <xacro:insert_block name="origin"/>
+        <mass value="${mass}" />
+        <inertia ixx="${(1/12) * mass * (3*radius*radius + length*length)}" ixy="0.0" ixz="0.0"
+                iyy="${(1/12) * mass * (3*radius*radius + length*length)}" iyz="0.0"
+                izz="${(1/2) * mass * (radius*radius)}" />
+    </inertial>
+  </xacro:macro>
+  <joint name="laser_joint" type="fixed">
+      <parent link="base_link"/>
+      <child link="laser_frame"/>
+      <origin xyz="-0.1 0 0.195" rpy="0 0 0"/>
+    </joint>
+    <link name="laser_frame">
+        <visual>
+            <geometry>
+                <cylinder radius="0.05" length="0.04"/>
+            </geometry>
+        </visual>
+        <visual>
+            <origin xyz="0 0 -0.05"/>
+            <geometry>
+                <cylinder radius="0.01" length="0.1"/>
+            </geometry>
+        </visual>
+        <collision>
+            <geometry>
+                <cylinder radius="0.05" length="0.04"/>
+            </geometry>
+        </collision>
+        <xacro:inertial_cylinder mass="0.1" length="0.04" radius="0.05">
+            <origin xyz="0 0 0" rpy="0 0 0"/>
+        </xacro:inertial_cylinder>
+    </link>
+    <gazebo reference="laser_frame">
+        <material>Gazebo/Red</material>
+        <sensor name="laser" type="ray">
+            <pose> 0 0 0 0 0 0 </pose>
+            <visualize>true</visualize>
+            <update_rate>10</update_rate>
+            <ray>
+                <scan>
+                    <horizontal>
+                        <samples>360</samples>
+                        <min_angle>-3.14</min_angle>
+                        <max_angle>3.14</max_angle>
+                    </horizontal>
+                </scan>
+                <range>
+                    <min>0.3</min>
+                    <max>10</max>
+                </range>
+            </ray>
+            <plugin name="laser_controller" filename="libgazebo_ros_ray_sensor.so">
+                <ros>
+                    <argument>~/out:=scan</argument>
+                </ros>
+                <output_type>sensor_msgs/LaserScan</output_type>
+                <frame_name>laser_frame</frame_name>
+            </plugin>
+        </sensor>
+    </gazebo>
+    <!-- SIMPLE CONTROLLER-->
+    <!-- <gazebo>
         <plugin name="diff_drive" filename="libgazebo_ros_diff_drive.so">
             <left_joint>wheel_1_joint</left_joint>
@@ -612,4 +677,47 @@
             <robot_base_frame>base_link</robot_base_frame>
         </plugin>
+      </gazebo> -->
+      <!-- ROS2 CONTROL-->
+      <ros2_control name="GazeboSystem" type="system">
+        <hardware>
+            <plugin>gazebo_ros2_control/GazeboSystem</plugin>
+        </hardware>
+        <joint name="wheel_1_joint">
+            <command_interface name="velocity">
+                <param name="min">-10</param>
+                <param name="max">10</param>
+            </command_interface>
+            <state_interface name="velocity"></state_interface>
+            <state_interface name="position"></state_interface>
+        </joint>
+        <joint name="wheel_4_joint">
+            <command_interface name="velocity">
+                <param name="min">-10</param>
+                <param name="max">10</param>
+            </command_interface>
+            <state_interface name="velocity"></state_interface>
+            <state_interface name="position"></state_interface>
+        </joint>
+        <joint name="wheel_3_joint">
+            <command_interface name="velocity">
+                <param name="min">-10</param>
+                <param name="max">10</param>
+            </command_interface>
+            <state_interface name="velocity"></state_interface>
+            <state_interface name="position"></state_interface>
+        </joint>
+        <joint name="wheel_6_joint">
+            <command_interface name="velocity">
+                <param name="min">-20</param>
+                <param name="max">20</param>
+            </command_interface>
+            <state_interface name="velocity"></state_interface>
+            <state_interface name="position"></state_interface>
+        </joint>
+      </ros2_control>
+      <gazebo>
+        <plugin name="gazebo_ros2_control" filename="libgazebo_ros2_control.so">
+            <parameters>/home/saieswaram/gujcost_rover/install/rover_description/share/rover_description/config/my_controllers.yaml</parameters>
+        </plugin>
       </gazebo>
 </robot>

Commit message: Add files via upload

File: src/rover_description/urdf/rover.urdf.xacro (robot description, xacro)
@@ -2,4 +2,10 @@
 <robot xmlns:xacro="http://www.ros.org/wiki/xacro" name="rover">
     <link name="base_link"></link>
+    <link name="base_footprint"></link>
+    <joint name="base_footprint_joint" type="fixed">
+        <origin rpy="0 0 0" xyz="0 0 0"></origin>
+        <parent link="base_link"></parent>
+        <child link="base_footprint"></child>
+    </joint>
     <link name="base_part_link">
         <inertial>
@@ -637,5 +643,5 @@
             <pose> 0 0 0 0 0 0 </pose>
             <visualize>true</visualize>
-            <update_rate>10</update_rate>
+            <update_rate>50</update_rate>
             <ray>
                 <scan>
@@ -661,5 +667,5 @@
     </gazebo>
     <!-- SIMPLE CONTROLLER-->
-    <!-- <gazebo>
+    <gazebo>
         <plugin name="diff_drive" filename="libgazebo_ros_diff_drive.so">
             <left_joint>wheel_1_joint</left_joint>
@@ -677,5 +683,5 @@
             <robot_base_frame>base_link</robot_base_frame>
         </plugin>
-      </gazebo> -->
+      </gazebo>
       <!-- ROS2 CONTROL-->
       <ros2_control name="GazeboSystem" type="system">
@@ -685,6 +691,6 @@
         <joint name="wheel_1_joint">
             <command_interface name="velocity">
-                <param name="min">-10</param>
-                <param name="max">10</param>
+                <param name="min">-20</param>
+                <param name="max">20</param>
             </command_interface>
             <state_interface name="velocity"></state_interface>
@@ -693,6 +699,6 @@
         <joint name="wheel_4_joint">
             <command_interface name="velocity">
-                <param name="min">-10</param>
-                <param name="max">10</param>
+                <param name="min">-20</param>
+                <param name="max">20</param>
             </command_interface>
             <state_interface name="velocity"></state_interface>
@@ -701,6 +707,6 @@
         <joint name="wheel_3_joint">
             <command_interface name="velocity">
-                <param name="min">-10</param>
-                <param name="max">10</param>
+                <param name="min">-20</param>
+                <param name="max">20</param>
             </command_interface>
             <state_interface name="velocity"></state_interface>
